File: RC_SHIELD/bb_power_motdrvs.kicad_sch (KiCad schematic)
At the start: 15 parts, among them J10 POWER_SUPPLY, J11 R_MOT_DRV, J12 Z_MOT_DRV, J13 PHI_MOT_DRV, J14 THETA_MOT_DRV

Commit message: added secondary MCU to schematic and made it more consistent
Parts:
- removed C4: 100nF, symbol Device:C
- removed C5: C, symbol Device:C
- removed C6, C7, C8: 1mF, symbol Device:C_Polarized
- removed D2: 3V3_STATUS, symbol Device:LED
- removed D3: 24V_STATUS, symbol Device:LED
- removed J10: POWER_SUPPLY, symbol Connector_Generic:Conn_01x04
- removed J11: R_MOT_DRV, symbol Connector_Generic:Conn_01x04
- removed J12: Z_MOT_DRV, symbol Connector_Generic:Conn_01x04
- removed J13: PHI_MOT_DRV, symbol Connector_Generic:Conn_01x04
- removed J14: THETA_MOT_DRV, symbol Connector_Generic:Conn_01x04
- removed R11: 1K, symbol Device:R
- removed R12: 20K, symbol Device:R
- removed VR1: LM3940IMP-3.3/NOPB, LM3940IMP-3.3/NOPB:VREG_LM3940IMP-3.3/NOPB, symbol LM3940IMP-3.3_NOPB:LM3940IMP-3.3/NOPB
Other:
- company: (none) -> LEGO Kör (legokor.hu)
