File: Aux_boards/Aux_boards.kicad_sch (KiCad schematic)
At the start: 0 parts

Commit message: added a resistor for test purposes
Parts:
- added R1: R, symbol Device:R
Changed lines of the file:
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@@
     (comment 1 "Design by Gergely Halász")
+  )
+  (symbol (lib_id "Device:R") (at 99.06 100.33 0) (unit 1)
+    (in_bom yes) (on_board yes) (dnp no) (fields_autoplaced)
+    (property "Reference" "R1" (at 101.6 99.695 0)
+      (effects (font (size 1.27 1.27)) (justify left))
+    )
+    (property "Value" "R" (at 101.6 102.235 0)
+      (effects (font (size 1.27 1.27)) (justify left))
+    )
+    (property "Footprint" "" (at 97.282 100.33 90)
+      (effects (font (size 1.27 1.27)) hide)
+    )
+    (property "Datasheet" "~" (at 99.06 100.33 0)
+      (effects (font (size 1.27 1.27)) hide)
+    )
+    (pin "1")
+    (pin "2")
+    (instances
+      (project "Aux_boards"
+        (path "/8cbd9868-8dda-4ab2-bfc7-d6cef0b3b037"
+          (reference "R1") (unit 1)
+        )
+      )
+    )
   )
   (sheet_instances
