File: Aux_boards/board2.kicad_sch (KiCad schematic)
At the start: 0 parts

Commit message: git test
Parts:
- added C1, C2: C, symbol Device:C
- added J1: DA15_Plug_MountingHoles, symbol Connector:DA15_Plug_MountingHoles
- added R1, R3, R5, R7: 220R, symbol Device:R
- added R10, R11, R9: 100R, symbol Device:R
- added R12, R13, R14, R15, R16, R17, R18: 100k, symbol Device:R
- added R2, R4, R6, R8: 10R, symbol Device:R
- added U1: ~, power_modules:DSN-1504-3A, symbol power_modules:DSN-1504-3A
- added U2: AMS1117-3.3, Package_TO_SOT_SMD:SOT-223-3_TabPin2, symbol Regulator_Linear:AMS1117-3.3
- added U3, U4, U5, U6, U7, U8, U9: SFH6345, SFH6345:DIP762W50P254L977H451Q8, symbol SFH6345:SFH6345
Connections:
- new net: R7.2, R8.1
- new net: R10.1, U9.3
- new net: R11.1, U8.3
- new net: R1.1, U6.3
- new net: R1.2, R2.1
- new net: R9.1, U7.3
- new net: R5.1, U4.3
- new net: R5.2, R6.1
- new net: R3.2, R4.1
- new net: R7.1, U5.3
- new net: R3.1, U3.3
- new net +24V: J1.15 (P15), J1.8, R12.1, U1.1 (Vin+), U1.2 (Vin+), U3.8, U4.8, U5.8, U6.8, U7.8, U8.8, U9.8
- new net +3.3V: C2.1, U2.2 (VO)
- new net +5V: C1.2, U1.7 (Vout+), U1.8 (Vout+), U2.3 (VI)
- new net GND: C1.1, C2.2, J1.0 (PAD), J1.10 (P10), J1.12 (P12), J1.14 (P14), J1.2, J1.4, J1.6, R10.2, R11.2, R2.2, R4.2, R6.2, R8.2, R9.2, U1.3 (Vin-), U1.4 (Vin-), U1.5 (Vout-), U1.6 (Vout-), U2.1 (GND), U3.5, U4.5, U5.5, U6.5, U7.5, U8.5, U9.5
- new net R_ENC_A: U5.2
- new net R_ENC_A_24: J1.3, U5.6
- new net R_ENC_B: U6.2
- new net R_ENC_B_24: J1.11 (P111), U6.6
- new net Z_ENC_A: U3.2
- new net Z_ENC_A_24: J1.1, R12.2, U3.6
- new net Z_ENC_B: U4.2
- new net Z_ENC_B_24: J1.9 (P9), U4.6
- new net Z_LIM_DN: U8.2
- new net Z_LIM_DN_24: J1.13 (P13), U8.6
- new net Z_LIM_UP: U7.2
- new net Z_LIM_UP_24: J1.5, U7.6
- new net Z_Pos: U9.2
- new net Z_Pos_24: J1.7, U9.6
