File: Aux_boards/board3.kicad_sch (KiCad schematic)
At the start: 0 parts

Commit message: dev
Parts:
- added C1, C2: 10 uF, symbol Device:C
- added C3: 47 uF, symbol Device:C
- added D1, D2, D3: LED, symbol Device:LED
- added J3: DE9_Plug_MountingHoles, symbol Connector:DE9_Plug_MountingHoles
- added J5: DB25_Plug_MountingHoles, symbol Connector:DB25_Plug_MountingHoles
- added R1, R2, R3: R, symbol Device:R
- added R15 (x6): 220R, symbol Device:R
- added R16 (x6): 10R, symbol Device:R
- added R17 (x6), R19 (x13): 100k, symbol Device:R
- added R18 (x13): 100R, symbol Device:R
- added U1: ~, power_modules:DSN-1504-3A, symbol power_modules:DSN-1504-3A
- added U2: AMS1117-3.3, Package_TO_SOT_SMD:SOT-223-3_TabPin2, symbol Regulator_Linear:AMS1117-3.3
- added U6 (x6), U7 (x13): SFH6345, SFH6345:SFH6345, symbol SFH6345:SFH6345
Connections:
- new net: R19.2, U7.6 (x5)
- new net: R15.2, U6.3 (x6)
- new net: R18.1, U7.3 (x13)
- new net: R15.1, R16.1 (x6)
- new net: D1.2 (A), R1.2
- new net: D3.2 (A), R3.2
- new net: D2.2 (A), R2.2
- new net +24V: J5.13, J5.25 (P25), R1.1, R17.1, R17.1, R17.1, R17.1, R17.1, R17.1, R19.1, R19.1, R19.1, R19.1, R19.1, R19.1, R19.1, R19.1, R19.1, R19.1, R19.1, R19.1, R19.1, U1.1 (Vin+), U1.2 (Vin+), U6.8, U6.8, U6.8, U6.8, U6.8, U6.8, U7.8, U7.8, U7.8, U7.8, U7.8, U7.8, U7.8, U7.8, U7.8, U7.8, U7.8, U7.8, U7.8
- new net +3.3V: C2.1, R3.1, U2.2 (VO)
- new net +5V: C1.1, C3.1, R2.1, U1.7 (Vout+), U1.8 (Vout+), U2.3 (VI)
- new net Alpha_ENC_A: U6.2
- new net Alpha_ENC_A_24: J5.3, R17.2, U6.6
- new net Alpha_ENC_B: U6.2
- new net Alpha_ENC_B_24: J5.16 (P16), R17.2, U6.6
- new net Alpha_LIM_1_24: J5.6, U7.2
- new net Alpha_LIM_2: U7.2
- new net Alpha_LIM_2_24: J5.19 (P19)
- new net Beta_ENC_A: U6.2
- new net Beta_ENC_A_24: J5.4, R17.2, U6.6
- new net Beta_ENC_B: U6.2
- new net Beta_ENC_B_24: J5.17 (P17), R17.2, U6.6
- new net Beta_LIM_1_24: J5.7, R19.2, U7.2, U7.6
- new net Beta_LIM_2: U7.2
- new net Beta_LIM_2_24: J5.20 (P20), R19.2, U7.6
- new net GND: C1.2, C2.2, C3.2, D1.1 (K), D2.1 (K), D3.1 (K), J5.0 (PAD), J5.11, J5.15 (P15), J5.18 (P18), J5.2, J5.21 (P21), J5.5, J5.8, R16.2, R16.2, R16.2, R16.2, R16.2, R16.2, R18.2, R18.2, R18.2, R18.2, R18.2, R18.2, R18.2, R18.2, R18.2, R18.2, R18.2, R18.2, R18.2, U1.3 (Vin-), U1.4 (Vin-), U1.5 (Vout-), U1.6 (Vout-), U2.1 (GND), U6.5, U6.5, U6.5, U6.5, U6.5, U6.5, U7.5, U7.5, U7.5, U7.5, U7.5, U7.5, U7.5, U7.5, U7.5, U7.5, U7.5, U7.5, U7.5
- new net R-Pos_24: J5.12, R19.2, U7.2, U7.6
- new net R_LIM_MAX: U7.2
- new net R_LIM_MAX_24: J5.23 (P23), R19.2, U7.6
- new net R_LIM_MIN_24: J5.10, R19.2, U7.2, U7.6
- new net Theta_ENC_A: U6.2
- new net Theta_ENC_A_24: J5.1, R17.2, U6.6
- new net Theta_ENC_B: U6.2
- new net Theta_ENC_B_24: J5.14 (P14), R17.2, U6.6
- new net Theta_LIM_CCW_24: J5.9, R19.2, U7.2, U7.6
- new net Theta_LIM_CLW: U7.2
- new net Theta_LIM_CLW_24: J5.22 (P22), R19.2, U7.6
- new net Theta_Pos_24: J5.24 (P24), R19.2, U7.2, U7.6

Commit message: commit message
Parts:
- removed R15 (x5): 220R, symbol Device:R
- removed R16 (x5): 10R, symbol Device:R
- removed R18 (x13): 100R, symbol Device:R
- added J10, J11, J12, J13, J14, J15, J16, J17, J18, J19, J20, J21, J25: Conn_01x03_Pin, symbol Connector:Conn_01x03_Pin
- added J22, J23, J24: Conn_01x04_Pin, symbol Connector:Conn_01x04_Pin
- added JP1, JP2, JP3: SolderJumper_3_Open, symbol Jumper:SolderJumper_3_Open
- added R15 (x16): 220R, symbol Device:R
- added R15 (x2): 100R, symbol Device:R
- added R16 (x21): 0R, symbol Device:R
- added R16 (x16): 10R, symbol Device:R
Connections:
- net +24V: now also JP1.3 (B), JP2.3 (B), JP3.3 (B)
- net +3.3V: now also J18.1 (Pin_1), J19.1 (Pin_1)
- net +5V: now also J3.2, J10.1 (Pin_1), J11.1 (Pin_1), J12.1 (Pin_1), J13.1 (Pin_1), J14.1 (Pin_1), J15.1 (Pin_1), J16.1 (Pin_1), J17.1 (Pin_1), J20.1 (Pin_1), J21.1 (Pin_1), J25.1 (Pin_1), JP1.1 (A), JP2.1 (A), JP3.1 (A)
- net Alpha_ENC_A: now also J23.2 (Pin_2)
- net Alpha_ENC_A_24: no longer R17.2, U6.6
- net Alpha_ENC_B: now also J23.3 (Pin_3)
- net Alpha_LIM_1_24: now also R19.2, U7.6; no longer U7.2
- net Alpha_LIM_2: now also J11.2 (Pin_2)
- net Alpha_LIM_2_24: now also R19.2, U7.6
- net Beta_ENC_A: now also J24.2 (Pin_2)
- net Beta_ENC_B: now also J24.3 (Pin_3)
- net Beta_LIM_1_24: no longer U7.2
- net Beta_LIM_2: now also J13.2 (Pin_2)
- net GND: now also J3.0 (PAD), J3.1, J10.3 (Pin_3), J11.3 (Pin_3), J12.3 (Pin_3), J13.3 (Pin_3), J14.3 (Pin_3), J15.3 (Pin_3), J16.3 (Pin_3), J17.3 (Pin_3), J18.3 (Pin_3), J19.3 (Pin_3), J20.3 (Pin_3), J21.3 (Pin_3), J22.4 (Pin_4), J23.4 (Pin_4), J24.4 (Pin_4), J25.3 (Pin_3), R16.2, R16.2, R16.2, R16.2, R16.2, R16.2, R16.2, R16.2, R16.2, R16.2, R16.2, R16.2, R16.2, R16.2, R16.2, R16.2, R16.2, R16.2, R16.2; no longer R16.2
- net R-Pos_24: no longer U7.2
- net R_LIM_MAX: now also J17.2 (Pin_2)
- net R_LIM_MIN_24: no longer U7.2
- net Theta_ENC_A: now also J22.2 (Pin_2)
- net Theta_ENC_B: now also J22.3 (Pin_3)
- net Theta_LIM_CCW_24: no longer U7.2
- net Theta_LIM_CLW: now also J15.2 (Pin_2)
- net Theta_Pos_24: no longer U7.2
- net EE_Srv_2_PWM_24: now reaches R19.2, U7.6
- net EE_Srv_2_PWM_24: now also J3.6
- net at U6.3: now also R15.2 (x5)
- net at U7.3: now also R15.2 (x13)
- net EE_Srv_1_PWM_24: now reaches J3.3
- net EE_Srv_1_PWM_24: now also R19.2, U7.6
- net Rx_1: now reaches J3.4
- net Tx_1: now reaches J3.5
- net EE_Srv_3_PWM_24: now reaches J3.7
- net EE_Srv_3_PWM_24: now also R19.2, U7.6
- net Rx_0: now reaches J3.8
- net Tx_0: now reaches J3.9
- net EE_Srv_3_PWM: now reaches U7.2
- net EE_Srv_3_PWM: now also J25.2 (Pin_2)
- net EE_Srv_1_PWM: now reaches U7.2
- net EE_Srv_1_PWM: now also J20.2 (Pin_2)
- net EE_Srv_2_PWM: now reaches U7.2
- net EE_Srv_2_PWM: now also J21.2 (Pin_2)
- new net: R16.1, R16.2 (x19)
- new net: R15.1, R16.1 (x18)
- new net: J22.1 (Pin_1), JP2.2 (C)
- new net: J23.1 (Pin_1), JP1.2 (C)
- new net: R17.2, U6.6
- new net: J24.1 (Pin_1), JP3.2 (C)
- new net Alpha_LIM_1: J10.2 (Pin_2), U7.2
- new net Beta_LIM_1: J12.2 (Pin_2), U7.2
- new net R-Pos: J19.2 (Pin_2), U7.2
- new net R_LIM_MIN: J16.2 (Pin_2), U7.2
- new net Theta_LIM_CCW: J14.2 (Pin_2), U7.2
- new net Theta_Pos: J18.2 (Pin_2), U7.2
Other:
- note added: "Optocouplers for Alpha, Beta, Theta Encoders"
- note added: "Optocouplers for Alpha, Beta, Theta, R Limit switches"
- note added: "Optocouplers for Servo motor 1-2-3"
- note added: "Optocouplers for Theta and R Position gates"
- note added: "Power Supply"
- moved on the sheet: C1, C2, C3, D1, D2, D3, J3, J5, R1, R15, R16, R17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

Commit message: updated aux board 3
Parts:
- added D2: LED, symbol Device:LED
- added R2: 5k1, symbol Device:R
- R1: value R -> 20k
- R15: value 220R -> 1k2
- R16: value 10R -> 180R
- R16: value 0R -> 33R
- R19: value 100k -> 1k
- R2: value R -> 5k1
- R3: value R -> 1k
Connections:
- net +24V: no longer R19.1, R19.1, R19.1, U7.8, U7.8, U7.8
- net +5V: now also R19.1, R19.1, R19.1, U7.8, U7.8, U7.8; no longer J3.2
- net GND: no longer J3.0 (PAD), J3.1
- net R-Pos renamed R_Pos
- net R-Pos_24 renamed R_Pos_24
- new net: D2.2 (A), R2.2
- new net +5VD: J3.2, R2.1
- new net GNDD: D2.1 (K), J3.0 (PAD), J3.1

Commit message: Removed unnecessary optocouplers
Parts:
- removed R15 (x14): 220R, symbol Device:R
- removed R15 (x3): 1k2, symbol Device:R
- removed R15 (x2): 100R, symbol Device:R
- removed R16 (x18): 0R, symbol Device:R
- removed R16 (x14): 10R, symbol Device:R
- removed R16 (x3): 180R, symbol Device:R
- removed R16 (x3): 33R, symbol Device:R
- removed R17 (x6), R19 (x10): 100k, symbol Device:R
- removed R19 (x3): 1k, symbol Device:R
- removed U6 (x6), U7 (x13): SFH6345, SFH6345:SFH6345, symbol SFH6345:SFH6345
- renumbered C1 to C4, C2 to C5, C3 to C6, D1 to D4, D2 to D5, D3 to D6, D2 to D7, R2 to R13, R1 to R20, R2 to R21, R3 to R22
Other:
- note removed: "Optocouplers for Alpha, Beta, Theta Encoders"
- note removed: "Optocouplers for Alpha, Beta, Theta, R Limit switches"
- note removed: "Optocouplers for Servo motor 1-2-3"
- note removed: "Optocouplers for Theta and R Position gates"
- company: (none) -> LEGO Kör (legokor.hu)
- title: (none) -> Karcsi (INDACT Robot Arm) - Auxiliary board 3
- moved on the sheet: C4, C5, C6, D4, D5, D6, D7, J12, J13, J14, J15, J16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
