File: Aux_board_1/Aux_board_1.kicad_sch (KiCad schematic)
At the start: 60 parts, among them J1 P03d, J2 P11a, J3 P10a, J4 PHI_ENC, J5 PHI_LIM_CLW, J6 PHI_LIM_CLW, J7 PHI_LIM_CLW, Q1 BSS138, Q10 BSS84, Q2 BSS84, Q3 BSS138, Q4 BSS84, Q5 BSS138, Q6 BSS84, Q7 BSS138, Q8 BSS84, Q9 BSS138, U2 AMS1117-3.3

Commit message: Started board 1 placement
Parts:
- C1, C2, C3, C4: footprint (none) -> Capacitor_SMD:C_0805_2012Metric_Pad1.18x1.45mm_HandSolder
- D1, D2, D3: footprint (none) -> LED_SMD:LED_0805_2012Metric_Pad1.15x1.40mm_HandSolder
- J1: footprint (none) -> Connector_Dsub:DSUB-37_Male_Horizontal_P2.77x2.84mm_EdgePinOffset7.70mm_Housed_MountingHolesOffset9.12mm
- J2: footprint (none) -> Connector_Dsub:DSUB-25_Female_Horizontal_P2.77x2.84mm_EdgePinOffset7.70mm_Housed_MountingHolesOffset9.12mm
- J3: footprint (none) -> Connector_Dsub:DSUB-15_Female_Horizontal_P2.77x2.84mm_EdgePinOffset7.70mm_Housed_MountingHolesOffset9.12mm
- J4: footprint (none) -> TerminalBlock_4Ucon:TerminalBlock_4Ucon_1x04_P3.50mm_Horizontal
- J5: footprint (none) -> Connector_PinSocket_2.54mm:PinSocket_1x03_P2.54mm_Vertical
- J6: value PHI_LIM_CLW -> PHI_LIM_CCW; footprint (none) -> Connector_PinSocket_2.54mm:PinSocket_1x03_P2.54mm_Vertical
- J7: value PHI_LIM_CLW -> PHI_HOME; footprint (none) -> Connector_PinSocket_2.54mm:PinSocket_1x03_P2.54mm_Vertical
- R1, R10, R11, R12, R13, R14, R15, R16, R17, R18, R19, R2, R20, R21, R22, R23, R24, R25, R26, R27, R28, R3, R30, R4, R5, R6, R7, R8, R9: footprint (none) -> Resistor_SMD:R_0805_2012Metric_Pad1.20x1.40mm_HandSolder
- R29: footprint (none) -> Resistor_SMD:R_0805_2012Metric_Pad1.20x1.40mm_HandSolder; now fitted
- TP1, TP2, TP3, TP4: footprint (none) -> TestPoint:TestPoint_Pad_2.0x2.0mm
Connections:
- net PHI_LIM_CCW_PWR: now reaches J6.1 (Pin_1), R25.2, R26.2, R27.2
- net PHI_LIM_CLW_PWR: now reaches J5.1 (Pin_1), R22.2, R23.2, R24.2
- net PHI_ENC_B_PG: now reaches Q3.3 (D), Q4.1 (G), R7.2
- net PHI_LIM_CCW_NG: now reaches Q7.1 (G), R14.1
- net PHI_LIM_CCW_PG: now reaches Q7.3 (D), Q8.1 (G), R13.2
- net PHI_ENC_A_PG: now reaches Q1.3 (D), Q2.1 (G), R4.2
- net PHI_ENC_PWR: now reaches J4.1 (Pin_1), R19.2, R20.2, R21.2
- net PHI_LIM_CLW_PG: now reaches Q5.3 (D), Q6.1 (G), R10.2
- net PHI_HOME_PWR: now reaches J7.1 (Pin_1), R28.2, R29.2, R30.2
- net PHIL_LIM_CLW_IN: now reaches J5.2 (Pin_2), R11.2
- net PHI_ENC_A_IN: now reaches J4.2 (Pin_2), R5.2
- net PHI_ENC_B_IN: now reaches J4.3 (Pin_3), R8.2
- net PHI_HOME_IN: now reaches J7.2 (Pin_2), R17.2
- net PHI_LIM_CLW_NG: now reaches Q5.1 (G), R11.1
- net PHI_LIM_CCW_IN: now reaches J6.2 (Pin_2), R14.2
- net PHI_HOME_PG: now reaches Q9.1 (G), R17.1
- net PHI_ENC_A_NG: now reaches Q1.1 (G), R5.1
- net PHI_ENC_B_NG: now reaches Q3.1 (G), R8.1
- net PHI_HOME_NG: now reaches Q10.1 (G), Q9.3 (D), R16.2

Commit message: Finished routing board 1
Connections:
- net +5V: now also U1.7 (Vout+)
Changed lines of the file:
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@@
+	)
+	(junction
+		(at 104.14 161.29)
+		(diameter 0)
+		(color 0 0 0 0)
 	)
 	(junction
@@
 	(wire
 		(pts
+			(xy 104.14 163.83) (xy 104.14 161.29)
+		)
+		(stroke
+			(width 0)
+			(type default)
+		)
+	)
+	(wire
+		(pts
 			(xy 64.77 73.66) (xy 64.77 76.2)
 		)
 		(stroke
+			(width 0)
+			(type default)
+		)
+	)
+	(wire
+		(pts
+			(xy 101.6 163.83) (xy 104.14 163.83)
+		)
+		(stroke

Commit message: Finished Board 2 schematic
Connections:
- net PHIL_LIM_CLW_IN renamed PHI_LIM_CLW_IN
Changed lines of the file:
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@@
 		)
 	)
-	(label "PHIL_LIM_CLW_IN"
+	(label "PHI_LIM_CLW_IN"
 		(at 123.19 111.76 90)
 		(fields_autoplaced yes)

Commit message: Filled out Board 1 BOM info
Parts:
- C1, C2, C3, C4: value 33u -> 47u; Supplier (none) -> Lomex; Supplier URL (none) -> https://lomex.hu/hu/webshop/#/search,82-11-74/stype,1; Supplier item no (none) -> 82-11-74
- D1, D2, D3: Supplier (none) -> DigiKey; Supplier URL (none) -> https://www.digikey.hu/hu/products/detail/harvatek-corporat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; Supplier item no (none) -> 3147-B1701NG--20D000314U1930CT-ND
- J1: Supplier (none) -> DigiKey; Supplier URL (none) -> https://www.digikey.hu/hu/products/detail/assmann-wsw-compo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; Supplier item no (none) -> AE10986-ND
- J2, J3: Supplier (none) -> LEGOlab; Supplier URL (none) -> -; Supplier item no (none) -> -
- J4: Supplier (none) -> Lomex; Supplier URL (none) -> https://lomex.hu/hu/webshop/#page,0/search,43-27-91/stype,1; Supplier item no (none) -> 43-27-91
- J5, J6, J7: Supplier (none) -> Lomex; Supplier URL (none) -> https://lomex.hu/hu/webshop/#page,0/search,43-03-71/stype,1; Supplier item no (none) -> 43-03-71
- Q1, Q3, Q5, Q7, Q9: value BSS138 -> BSS138KJ; Supplier (none) -> Lomex; Supplier URL (none) -> https://lomex.hu/hu/webshop/#page,0/search,86-07-11/stype,1; Supplier item no (none) -> 86-07-11
- Q10, Q2, Q4, Q6, Q8: value BSS84 -> BSS84KJ
- R1: Supplier (none) -> Lomex; Supplier URL (none) -> https://lomex.hu/hu/webshop/#page,0/search,81-10-91/stype,1; Supplier item no (none) -> 81-10-91
- R10, R12, R13, R15, R16, R18, R4, R6, R7, R9: Supplier (none) -> Lomex; Supplier item no (none) -> 81-10-84
- R11, R14, R17, R5, R8: Supplier (none) -> Lomex; Supplier item no (none) -> 81-10-95
- R19, R20, R21, R22, R23, R24, R25, R26, R27, R28, R29, R30: Supplier (none) -> LCSC; Supplier URL (none) -> https://www.lcsc.com/product-detail/Chip-Resistor-Surface-M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; Supplier item no (none) -> C304192
- R2: Supplier (none) -> Lomex; Supplier item no (none) -> 81-10-81
- R3: Supplier (none) -> Lomex; Supplier item no (none) -> 81-10-77
- TP1, TP2, TP3, TP4: Supplier (none) -> -; Supplier URL (none) -> -; Supplier item no (none) -> -
- U1: value ~ -> DSN-1504-3A; Supplier (none) -> Hestore; Supplier URL (none) -> https://www.hestore.hu/prod_10038118.html; Supplier item no (none) -> 100.381.18
- U2: Supplier (none) -> LCSC; Supplier URL (none) -> https://www.lcsc.com/product-detail/Linear-Voltage-Regulato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; Supplier item no (none) -> C6186

Commit message: Finished Board 2 layout
Parts:
- C1, C2, C3, C4, R19, R20, R21, R22, R23, R24, R25, R26, R27, R28, R29, R30, U1, U2: Sourced (none) -> 0
- D1, D2, D3, J1, J2, J3, J4, J5, J6, J7, Q1, Q3, Q5, Q7, Q9, R1, R10, R11, R12, R13, R14, R15, R16, R17, R18, R2, R3, R4, R5, R6, R7, R8, R9: Sourced (none) -> 1
- Q10, Q2, Q4, Q6, Q8: Sourced (none) -> 0; Supplier (none) -> Lomex; Supplier URL (none) -> https://lomex.hu/hu/webshop/#page,0/search,86-07-17/stype,1; Supplier item no (none) -> 86-07-17
- TP1, TP2, TP3, TP4: Sourced (none) -> -
