File: Aux_board_1/Aux_board_1.kicad_pcb (KiCad board)
At the start: 2 copper layers, 100 x 84.1 mm, 52 parts, among them J1 PWR OUT & TP, J10 P11a, J11 P03d, J2 ENC PWR SEL, J3 LIM PWR SEL, J4 HOM PWR SEL, J5 PHI_ENC, J6 PHI_LIM_CLW, J7 PHI_LIM_CCW, J8 PHI_HOME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

Commit message: Aux Board 1 finished and prod-plotted
Parts:
- moved Q5 28.2 mm to (115.2, 93.8)
- moved C4 28.2 mm to (74.8, 121.6)
- moved J1 28.2 mm to (87.5, 121.1)
- moved J4 28.2 mm to (103.8, 128.0)
- moved Q2 28.2 mm to (93.0, 92.9)
- moved Q3 28.2 mm to (116.2, 81.0)
- moved R10 28.2 mm to (118.2, 90.7)
- moved R12 28.2 mm to (106.2, 102.7)
- moved R3 28.2 mm to (77.5, 117.1)
- moved R4 28.2 mm to (105.1, 92.9)
- moved R5 28.2 mm to (97.4, 92.9)
- moved R6 28.2 mm to (88.9, 92.9)
- moved R9 28.2 mm to (107.3, 89.9)
- moved U2 28.2 mm to (74.8, 127.1)
- moved C2 28.2 mm to (82.3, 125.3)
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Other:
- board text added: "0"
- board text added: "0 mm"
- board text added: "0,015 mm"
- board text added: "0,02"
- board text added: "0,035 mm"
- board text added: "1"
- board text added: "1,51 mm"
- board text added: "3,8"
- board text added: "4,5"
- board text added: "A"
- board text added: "B"
- board text added: "B.Cu"
- board text added: "B.Mask"
- board text added: "B.Paste"
- board text added: "B.Silkscreen"
- board text added: "Bottom Silk Screen"
- board text added: "Bottom Solder Mask"
- board text added: "Bottom Solder Paste"
- board text added: "Color"
- board text added: "Dielectric"
- board text added: "Direct Printing"
- board text added: "Epsilon R"
- board text added: "F.Cu"
- board text added: "F.Mask"
- board text added: "F.Paste"
- board text added: "F.Silkscreen"
- board text added: "FR4"
- board text added: "FR4 natural"
- board text added: "GND"
- board text added: "Green"
- board text added: "Layer Name"
- board text added: "Liquid Ink"
- board text added: "Loss Tangent"
- board text added: "Material"
- board text added: "PHI ENCODER"
- board text added: "PHI LIMIT ↺ GND SIG PWR"
- board text added: "PHI LIMIT ↻"
- board text added: "PWR"
- board text added: "SIG"
- board text added: "Thickness (mm)"
- board text added: "Top Silk Screen"
- board text added: "Top Solder Mask"
- board text added: "Top Solder Paste"
- board text added: "Type"
- board text added: "White"
- board text added: "copper"
- board text added: "core"
