File: Aux_board_2/Aux_board_2.kicad_pcb (KiCad board)
At the start: 2 copper layers, 72 parts, among them J1 P10d, J2 R_ENC, J3 Z_ENC, J4 Z_LIM_UP, J5 Z_LIM_DN, J6 Z_HOME, Q1 BSS138, Q10 BSS84, Q11 BSS138, Q12 BSS84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

Commit message: Finished Board 2 layout
Parts:
- removed J5: Z_LIM_DN, Connector_PinHeader_2.54mm:PinHeader_1x03_P2.54mm_Horizontal
- removed J6: Z_HOME, Connector_PinHeader_2.54mm:PinHeader_1x03_P2.54mm_Horizontal
- added REF**: INDACTlogo, LEGOkor:INDACTlogoSmall, F.Cu at (135.9, 106.3)
- added REF**: LEGOkorLogo, LEGOkor:LEGOkorLogoSmall, F.Cu at (124.7, 103.2)
- added REF**: MountingHole_3mm, MountingHole:MountingHole_3mm, F.Cu at (127.7, 107.8)
- added REF**: MountingHole_3mm, MountingHole:MountingHole_3mm, F.Cu at (127.7, 66.0)
- C1, C2, C3, C4: value 33u -> 47u
- J1, R16, R17, R18, R28, R29, R30, R34, R35, R36: moved to B.Cu
- J2: value R_ENC -> Z_LIM_DN | R_ENC; footprint Connector_PinHeader_2.54mm:PinHeader_1x04_P2.54mm_Horizontal -> Connector_PinHeader_2.54mm:PinHeader_2x04_P2.54mm_Horizontal
- J3: value Z_ENC -> Z_ENC | Z_LIM_UP; footprint Connector_PinHeader_2.54mm:PinHeader_1x04_P2.54mm_Horizontal -> Connector_PinHeader_2.54mm:PinHeader_2x04_P2.54mm_Horizontal; moved to B.Cu
- J4: value Z_LIM_UP -> Z_HOME; moved to B.Cu
- Q1, Q3, Q5, Q9: value BSS138 -> BSS138KJ
- Q10, Q2, Q4, Q6: value BSS84 -> BSS84KJ
- Q11, Q13, Q7: value BSS138 -> BSS138KJ; moved to B.Cu
- Q12, Q14, Q8: value BSS84 -> BSS84KJ; moved to B.Cu
- U1: value ~ -> DSN-1504-3A
- moved Q8 163.0 mm to (116.8, 68.7), turned to 90 degrees
- moved Q6 161.6 mm to (116.8, 64.0), turned to -90 degrees
- moved R15 149.3 mm to (112.4, 64.0), turned to 90 degrees
- moved Q5 147.7 mm to (134.0, 64.0), turned to -90 degrees
- moved R18 146.6 mm to (112.4, 68.7), turned to 90 degrees
- moved Q7 145.2 mm to (134.0, 68.7), turned to 90 degrees
- moved R14 140.0 mm to (121.2, 64.0), turned to 90 degrees
- moved Q12 139.2 mm to (138.0, 100.6)
- moved Q11 138.5 mm to (138.0, 109.0)
- moved R17 137.3 mm to (121.2, 68.7), turned to -90 degrees
- moved Q14 131.2 mm to (147.4, 100.6)
- moved Q13 129.5 mm to (147.5, 109.0)
- moved Q9 128.3 mm to (152.1, 77.4)
- moved Q10 126.7 mm to (152.1, 86.6)
- moved R16 125.0 mm to (138.8, 68.7), turned to -90 degrees
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Connections:
- J2 pad 1: /R_ENC_PWR -> GND
- J2 pad 2: /R_ENC_A_IN -> GND
- J2 pad 3: /R_ENC_B_IN -> /Z_LIM_DN_IN
- J2 pad 4: GND -> /R_ENC_B_IN
- J3 pad 1: /Z_ENC_PWR -> GND
- J3 pad 2: /Z_ENC_A_IN -> GND
- J3 pad 4: GND -> /Z_LIM_UP_IN
- J4 pad 1: /Z_LIM_UP_PWR -> /Z_HOME_PWR
- J4 pad 2: /Z_LIM_UP_IN -> /Z_HOME_IN
- Q13 pad 1: /Z_HOME_PG -> /Z_HOME_NG
- Q13 pad 3: /Z_HOME_NG -> /Z_HOME_PG
- Q14 pad 1: /Z_HOME_NG -> /Z_HOME_PG
- R34 pad 1: /Z_HOME_PG -> /Z_HOME_NG
- R35 pad 2: /Z_HOME_NG -> /Z_HOME_PG
Routing:
- net GND: track 119.7 -> 377.5 mm, vias 3 -> 70
- net /Z_HOME: track 0.00 -> 108.5 mm
- net /Z_ENC_A: track 0.00 -> 101.5 mm, vias 0 -> 1
- net /R_ENC_B: track 0.00 -> 101.2 mm, vias 0 -> 1
- net /Z_ENC_B: track 0.00 -> 85.4 mm
- net /R_ENC_A: track 5.03 -> 89.4 mm, vias 0 -> 1
- net /Z_LIM_UP: track 0.00 -> 69.2 mm, vias 0 -> 5
- net +24V: track 133.6 -> 184.6 mm, vias 0 -> 7
- net /Z_LIM_DN: track 0.00 -> 41.7 mm, vias 0 -> 1
- net /Z_HOME_PWR: track 39.0 -> 69.7 mm, vias 0 -> 4
- net +5V: track 101.0 -> 79.3 mm
- net /Z_ENC_B_PG: track 0.00 -> 20.2 mm
- net /Z_ENC_A_PG: track 0.00 -> 17.8 mm
- net /Z_LIM_DN_IN: track 0.00 -> 17.0 mm
- net /Z_HOME_IN: track 0.00 -> 16.3 mm
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- added copper zone on B.Cu, net GND
- added copper zone on F.Cu, net GND
Other:
- board outline added: 56.4 x 70.5 mm
- board text added: "/------- Z HOME : GND | HOM | PWR / /----- R ENC : GND | B | A | PWR / / /--- Z LIM ↓: GND | LIM | x | PWR"
- board text added: "24V"
- board text added: "24V_|______|_______|______|"
- board text added: "3.3V"
- board text added: "3.3V_|______|_______|______|_______|"
- board text added: "5V"
- board text added: "5V__|______|_______|______|_______|"
- board text added: "GND"
- board text added: "GND LIM x PWR GND B A PWR"
- board text added: "Karcsi - Aux. Board 2"
- board text added: "Rev. 1.0"
- board text added: "Set supply voltage with 0Ω resistors"
- board text added: "TO AUX. BOARD 1"
- board text added: "Z ↑ Z ENC"
- board text added: "Z ↑ | Z ENC | Z HOM | R ENC | Z ↓"

Commit message: Initialized Board 3 project
Parts:
- turned TP2 to 90 degrees
