File: Aux_board_3/Aux_board_3.kicad_pcb (KiCad board)
At the start: 2 copper layers, 0 parts

Commit message: Board 3 layout started
Parts:
- added C1: 47u, Capacitor_SMD:C_0805_2012Metric_Pad1.18x1.45mm_HandSolder, F.Cu at (221.1, 89.9)
- added C2: 47u, Capacitor_SMD:C_0805_2012Metric_Pad1.18x1.45mm_HandSolder, F.Cu at (221.1, 92.9)
- added C3: 47u, Capacitor_SMD:C_0805_2012Metric_Pad1.18x1.45mm_HandSolder, F.Cu at (221.1, 95.9)
- added C4: 47u, Capacitor_SMD:C_0805_2012Metric_Pad1.18x1.45mm_HandSolder, F.Cu at (221.1, 98.9)
- added C5: 47u, Capacitor_SMD:C_0805_2012Metric_Pad1.18x1.45mm_HandSolder, F.Cu at (197.3, 134.3)
- added C6: 1n5, Capacitor_SMD:C_0805_2012Metric_Pad1.18x1.45mm_HandSolder, F.Cu at (197.3, 137.3)
- added C7: 1n5, Capacitor_SMD:C_0805_2012Metric_Pad1.18x1.45mm_HandSolder, F.Cu at (197.3, 140.4)
- added D1: LED_G, LED_SMD:LED_0805_2012Metric_Pad1.15x1.40mm_HandSolder, F.Cu at (235.4, 86.4)
- added D2: LED_G, LED_SMD:LED_0805_2012Metric_Pad1.15x1.40mm_HandSolder, F.Cu at (235.4, 89.4)
- added D3: LED_G, LED_SMD:LED_0805_2012Metric_Pad1.15x1.40mm_HandSolder, F.Cu at (235.4, 92.5)
- added D4: LED_G, LED_SMD:LED_0805_2012Metric_Pad1.15x1.40mm_HandSolder, F.Cu at (215.2, 134.3)
- added J1: P11d, Connector_Dsub:DSUB-25_Male_Horizontal_P2.77x2.84mm_EdgePinOffset7.70mm_Housed_MountingHolesOffset9.12mm, F.Cu at (66.3, 52.8)
- added J10: R_HOME, Connector_PinHeader_2.54mm:PinHeader_1x03_P2.54mm_Horizontal, F.Cu at (203.6, 78.9)
- added J11: R_LIM_MAX, Connector_PinHeader_2.54mm:PinHeader_1x03_P2.54mm_Horizontal, F.Cu at (203.6, 88.6)
- added J2: P04d, Connector_Dsub:DSUB-9_Male_Horizontal_P2.77x2.84mm_EdgePinOffset7.70mm_Housed_MountingHolesOffset9.12mm, F.Cu at (66.2, 19.7)
- added J3: MODBUS, Connector_PinHeader_1.00mm:PinHeader_1x04_P1.00mm_Horizontal, F.Cu at (205.3, 140.8)
- added J4: ~, Connector_PinHeader_2.54mm:PinHeader_2x04_P2.54mm_Horizontal, F.Cu at (187.6, 38.4)
- added J5: ~, Connector_PinHeader_2.54mm:PinHeader_2x04_P2.54mm_Horizontal, F.Cu at (187.6, 50.6)
- added J6: ~, Connector_PinHeader_2.54mm:PinHeader_2x04_P2.54mm_Horizontal, F.Cu at (187.6, 62.9)
- added J7: ~, Connector_PinHeader_2.54mm:PinHeader_2x04_P2.54mm_Horizontal, F.Cu at (187.6, 75.1)
- added J8: ~, Connector_PinHeader_2.54mm:PinHeader_2x04_P2.54mm_Horizontal, F.Cu at (187.6, 87.4)
- added J9: ~, Connector_PinHeader_2.54mm:PinHeader_2x04_P2.54mm_Horizontal, F.Cu at (187.6, 99.6)
- added Q1: BSS138KJ, Package_TO_SOT_SMD:SOT-23, F.Cu at (260.9, 38.5)
- added Q10: BSS84KJ, Package_TO_SOT_SMD:SOT-23, F.Cu at (270.7, 43.1)
- added Q11: BSS138KJ, Package_TO_SOT_SMD:SOT-23, F.Cu at (270.7, 47.7)
- added Q12: BSS84KJ, Package_TO_SOT_SMD:SOT-23, F.Cu at (270.7, 52.3)
- added Q13: BSS138KJ, Package_TO_SOT_SMD:SOT-23, F.Cu at (275.6, 38.5)
- added Q14: BSS84KJ, Package_TO_SOT_SMD:SOT-23, F.Cu at (275.6, 43.1)
- added Q15: BSS138KJ, Package_TO_SOT_SMD:SOT-23, F.Cu at (275.6, 47.7)
- added Q16: BSS84KJ, Package_TO_SOT_SMD:SOT-23, F.Cu at (275.6, 52.3)
- added Q17: BSS138KJ, Package_TO_SOT_SMD:SOT-23, F.Cu at (260.9, 76.7)
- added Q18: BSS84KJ, Package_TO_SOT_SMD:SOT-23, F.Cu at (260.9, 81.3)
- added Q19: BSS138KJ, Package_TO_SOT_SMD:SOT-23, F.Cu at (260.9, 85.9)
- added Q2: BSS84KJ, Package_TO_SOT_SMD:SOT-23, F.Cu at (260.9, 43.1)
- added Q20: BSS84KJ, Package_TO_SOT_SMD:SOT-23, F.Cu at (260.9, 90.5)
- added Q21: BSS138KJ, Package_TO_SOT_SMD:SOT-23, F.Cu at (265.8, 76.7)
- added Q22: BSS84KJ, Package_TO_SOT_SMD:SOT-23, F.Cu at (265.8, 81.3)
- added Q23: BSS138KJ, Package_TO_SOT_SMD:SOT-23, F.Cu at (265.8, 85.9)
- added Q24: BSS84KJ, Package_TO_SOT_SMD:SOT-23, F.Cu at (265.8, 90.5)
- added Q25: BSS138KJ, Package_TO_SOT_SMD:SOT-23, F.Cu at (270.7, 76.7)
- added Q26: BSS84KJ, Package_TO_SOT_SMD:SOT-23, F.Cu at (270.7, 81.3)
- added Q27: BSS138KJ, Package_TO_SOT_SMD:SOT-23, F.Cu at (270.7, 85.9)
- added Q28: BSS84KJ, Package_TO_SOT_SMD:SOT-23, F.Cu at (270.7, 90.5)
- added Q29: BSS138KJ, Package_TO_SOT_SMD:SOT-23, F.Cu at (275.6, 76.7)
- added Q3: BSS138KJ, Package_TO_SOT_SMD:SOT-23, F.Cu at (260.9, 47.7)
- added Q30: BSS84KJ, Package_TO_SOT_SMD:SOT-23, F.Cu at (275.6, 81.3)
- added Q31: BSS138KJ, Package_TO_SOT_SMD:SOT-23, F.Cu at (275.6, 85.9)
- added Q32: BSS84KJ, Package_TO_SOT_SMD:SOT-23, F.Cu at (275.6, 90.5)
- added Q33: BSS138KJ, Package_TO_SOT_SMD:SOT-23, F.Cu at (192.5, 135.2)
- added Q34: BSS138KJ, Package_TO_SOT_SMD:SOT-23, F.Cu at (192.5, 139.9)
- added Q35: BSS138KJ, Package_TO_SOT_SMD:SOT-23, F.Cu at (192.5, 144.5)
- added Q4: BSS84KJ, Package_TO_SOT_SMD:SOT-23, F.Cu at (260.9, 52.3)
- added Q5: BSS138KJ, Package_TO_SOT_SMD:SOT-23, F.Cu at (265.8, 38.5)
- added Q6: BSS84KJ, Package_TO_SOT_SMD:SOT-23, F.Cu at (265.8, 43.1)
- added Q7: BSS138KJ, Package_TO_SOT_SMD:SOT-23, F.Cu at (265.8, 47.7)
- added Q8: BSS84KJ, Package_TO_SOT_SMD:SOT-23, F.Cu at (265.8, 52.3)
- added Q9: BSS138KJ, Package_TO_SOT_SMD:SOT-23, F.Cu at (270.7, 38.5)
- added R1: 2k2, Resistor_SMD:R_0805_2012Metric_Pad1.20x1.40mm_HandSolder, F.Cu at (221.1, 78.0)
- added R10: 560R, Resistor_SMD:R_0805_2012Metric_Pad1.20x1.40mm_HandSolder, F.Cu at (187.7, 130.7)
- added R11: 560R, Resistor_SMD:R_0805_2012Metric_Pad1.20x1.40mm_HandSolder, F.Cu at (187.7, 133.7)
- added R12: 560R, Resistor_SMD:R_0805_2012Metric_Pad1.20x1.40mm_HandSolder, F.Cu at (187.7, 136.6)
- added R13: 0R, Resistor_SMD:R_0805_2012Metric_Pad1.20x1.40mm_HandSolder, F.Cu at (221.1, 86.9)
- added R14: 0R, Resistor_SMD:R_0805_2012Metric_Pad1.20x1.40mm_HandSolder, F.Cu at (225.8, 78.0)
- added R15: 0R, Resistor_SMD:R_0805_2012Metric_Pad1.20x1.40mm_HandSolder, F.Cu at (225.8, 81.0)
- added R16: 0R, Resistor_SMD:R_0805_2012Metric_Pad1.20x1.40mm_HandSolder, F.Cu at (225.8, 83.9)
- added R17: 0R, Resistor_SMD:R_0805_2012Metric_Pad1.20x1.40mm_HandSolder, F.Cu at (225.8, 86.9)
- added R18: 0R, Resistor_SMD:R_0805_2012Metric_Pad1.20x1.40mm_HandSolder, F.Cu at (230.6, 78.0)
- added R19: 0R, Resistor_SMD:R_0805_2012Metric_Pad1.20x1.40mm_HandSolder, F.Cu at (230.6, 81.0)
- added R2: 330R, Resistor_SMD:R_0805_2012Metric_Pad1.20x1.40mm_HandSolder, F.Cu at (221.1, 81.0)
- added R20: 0R, Resistor_SMD:R_0805_2012Metric_Pad1.20x1.40mm_HandSolder, F.Cu at (230.6, 83.9)
- added R21: 0R, Resistor_SMD:R_0805_2012Metric_Pad1.20x1.40mm_HandSolder, F.Cu at (230.6, 86.9)
- added R22: 4k7, Resistor_SMD:R_0805_2012Metric_Pad1.20x1.40mm_HandSolder, F.Cu at (260.8, 56.0)
- added R23: 560R, Resistor_SMD:R_0805_2012Metric_Pad1.20x1.40mm_HandSolder, F.Cu at (260.8, 59.0)
- added R24: 560R, Resistor_SMD:R_0805_2012Metric_Pad1.20x1.40mm_HandSolder, F.Cu at (260.8, 61.9)
- added R25: 4k7, Resistor_SMD:R_0805_2012Metric_Pad1.20x1.40mm_HandSolder, F.Cu at (260.8, 64.9)
- added R26: 560R, Resistor_SMD:R_0805_2012Metric_Pad1.20x1.40mm_HandSolder, F.Cu at (260.8, 67.8)
- added R27: 560R, Resistor_SMD:R_0805_2012Metric_Pad1.20x1.40mm_HandSolder, F.Cu at (260.8, 70.8)
- added R28: 4k7, Resistor_SMD:R_0805_2012Metric_Pad1.20x1.40mm_HandSolder, F.Cu at (265.6, 56.0)
- added R29: 560R, Resistor_SMD:R_0805_2012Metric_Pad1.20x1.40mm_HandSolder, F.Cu at (265.6, 59.0)
- added R3: 150R, Resistor_SMD:R_0805_2012Metric_Pad1.20x1.40mm_HandSolder, F.Cu at (221.1, 83.9)
- added R30: 560R, Resistor_SMD:R_0805_2012Metric_Pad1.20x1.40mm_HandSolder, F.Cu at (265.6, 61.9)
- added R31: 4k7, Resistor_SMD:R_0805_2012Metric_Pad1.20x1.40mm_HandSolder, F.Cu at (265.6, 64.9)
- added R32: 560R, Resistor_SMD:R_0805_2012Metric_Pad1.20x1.40mm_HandSolder, F.Cu at (265.6, 67.8)
- added R33: 560R, Resistor_SMD:R_0805_2012Metric_Pad1.20x1.40mm_HandSolder, F.Cu at (265.6, 70.8)
- added R34: 4k7, Resistor_SMD:R_0805_2012Metric_Pad1.20x1.40mm_HandSolder, F.Cu at (270.3, 56.0)
- added R35: 560R, Resistor_SMD:R_0805_2012Metric_Pad1.20x1.40mm_HandSolder, F.Cu at (270.3, 59.0)
- added R36: 560R, Resistor_SMD:R_0805_2012Metric_Pad1.20x1.40mm_HandSolder, F.Cu at (270.3, 61.9)
- added R37: 4k7, Resistor_SMD:R_0805_2012Metric_Pad1.20x1.40mm_HandSolder, F.Cu at (270.3, 64.9)
- added R38: 560R, Resistor_SMD:R_0805_2012Metric_Pad1.20x1.40mm_HandSolder, F.Cu at (270.3, 67.8)
- added R39: 560R, Resistor_SMD:R_0805_2012Metric_Pad1.20x1.40mm_HandSolder, F.Cu at (270.3, 70.8)
- added R4: 330R, Resistor_SMD:R_0805_2012Metric_Pad1.20x1.40mm_HandSolder, F.Cu at (187.7, 113.0)
- added R40: 4k7, Resistor_SMD:R_0805_2012Metric_Pad1.20x1.40mm_HandSolder, F.Cu at (275.1, 56.0)
- added R41: 560R, Resistor_SMD:R_0805_2012Metric_Pad1.20x1.40mm_HandSolder, F.Cu at (275.1, 59.0)
- added R42: 560R, Resistor_SMD:R_0805_2012Metric_Pad1.20x1.40mm_HandSolder, F.Cu at (275.1, 61.9)
- added R43: 4k7, Resistor_SMD:R_0805_2012Metric_Pad1.20x1.40mm_HandSolder, F.Cu at (275.1, 64.9)
- added R44: 560R, Resistor_SMD:R_0805_2012Metric_Pad1.20x1.40mm_HandSolder, F.Cu at (275.1, 67.8)
- added R45: 560R, Resistor_SMD:R_0805_2012Metric_Pad1.20x1.40mm_HandSolder, F.Cu at (275.1, 70.8)
- added R46: 4k7, Resistor_SMD:R_0805_2012Metric_Pad1.20x1.40mm_HandSolder, F.Cu at (260.8, 94.2)
- added R47: 560R, Resistor_SMD:R_0805_2012Metric_Pad1.20x1.40mm_HandSolder, F.Cu at (260.8, 97.2)
- added R48: 560R, Resistor_SMD:R_0805_2012Metric_Pad1.20x1.40mm_HandSolder, F.Cu at (260.8, 100.1)
- added R49: 4k7, Resistor_SMD:R_0805_2012Metric_Pad1.20x1.40mm_HandSolder, F.Cu at (260.8, 103.1)
- added R5: 120R, Resistor_SMD:R_0805_2012Metric_Pad1.20x1.40mm_HandSolder, F.Cu at (187.7, 116.0)
- added R50: 560R, Resistor_SMD:R_0805_2012Metric_Pad1.20x1.40mm_HandSolder, F.Cu at (260.8, 106.0)
- added R51: 560R, Resistor_SMD:R_0805_2012Metric_Pad1.20x1.40mm_HandSolder, F.Cu at (260.8, 109.0)
- added R52: 4k7, Resistor_SMD:R_0805_2012Metric_Pad1.20x1.40mm_HandSolder, F.Cu at (265.6, 94.2)
- added R53: 560R, Resistor_SMD:R_0805_2012Metric_Pad1.20x1.40mm_HandSolder, F.Cu at (265.6, 97.2)
- added R54: 560R, Resistor_SMD:R_0805_2012Metric_Pad1.20x1.40mm_HandSolder, F.Cu at (265.6, 100.1)
- added R55: 4k7, Resistor_SMD:R_0805_2012Metric_Pad1.20x1.40mm_HandSolder, F.Cu at (265.6, 103.1)
- added R56: 560R, Resistor_SMD:R_0805_2012Metric_Pad1.20x1.40mm_HandSolder, F.Cu at (265.6, 106.0)
- added R57: 560R, Resistor_SMD:R_0805_2012Metric_Pad1.20x1.40mm_HandSolder, F.Cu at (265.6, 109.0)
- added R58: 4k7, Resistor_SMD:R_0805_2012Metric_Pad1.20x1.40mm_HandSolder, F.Cu at (270.3, 94.2)
- added R59: 560R, Resistor_SMD:R_0805_2012Metric_Pad1.20x1.40mm_HandSolder, F.Cu at (270.3, 97.2)
- added R6: 120R, Resistor_SMD:R_0805_2012Metric_Pad1.20x1.40mm_HandSolder, F.Cu at (187.7, 118.9)
- added R60: 560R, Resistor_SMD:R_0805_2012Metric_Pad1.20x1.40mm_HandSolder, F.Cu at (270.3, 100.1)
- added R61: 4k7, Resistor_SMD:R_0805_2012Metric_Pad1.20x1.40mm_HandSolder, F.Cu at (270.3, 103.1)
- added R62: 560R, Resistor_SMD:R_0805_2012Metric_Pad1.20x1.40mm_HandSolder, F.Cu at (270.3, 106.0)
- added R63: 560R, Resistor_SMD:R_0805_2012Metric_Pad1.20x1.40mm_HandSolder, F.Cu at (270.3, 109.0)
- added R64: 4k7, Resistor_SMD:R_0805_2012Metric_Pad1.20x1.40mm_HandSolder, F.Cu at (275.1, 94.2)
- added R65: 560R, Resistor_SMD:R_0805_2012Metric_Pad1.20x1.40mm_HandSolder, F.Cu at (275.1, 97.2)
- added R66: 560R, Resistor_SMD:R_0805_2012Metric_Pad1.20x1.40mm_HandSolder, F.Cu at (275.1, 100.1)
- added R67: 4k7, Resistor_SMD:R_0805_2012Metric_Pad1.20x1.40mm_HandSolder, F.Cu at (275.1, 103.1)
- added R68: 560R, Resistor_SMD:R_0805_2012Metric_Pad1.20x1.40mm_HandSolder, F.Cu at (275.1, 106.0)
- added R69: 560R, Resistor_SMD:R_0805_2012Metric_Pad1.20x1.40mm_HandSolder, F.Cu at (275.1, 109.0)
- added R7: 560R, Resistor_SMD:R_0805_2012Metric_Pad1.20x1.40mm_HandSolder, F.Cu at (187.7, 121.9)
- added R8: 560R, Resistor_SMD:R_0805_2012Metric_Pad1.20x1.40mm_HandSolder, F.Cu at (187.7, 124.8)
- added R9: 560R, Resistor_SMD:R_0805_2012Metric_Pad1.20x1.40mm_HandSolder, F.Cu at (187.7, 127.8)
- added TP1: GND, TestPoint:TestPoint_Pad_2.0x2.0mm, F.Cu at (216.7, 78.6)
- added TP2: 24V, TestPoint:TestPoint_Pad_2.0x2.0mm, F.Cu at (216.7, 82.6)
- added TP3: 5V, TestPoint:TestPoint_Pad_2.0x2.0mm, F.Cu at (216.7, 86.7)
- added TP4: 3V3, TestPoint:TestPoint_Pad_2.0x2.0mm, F.Cu at (216.7, 90.7)
- added TP5: 5V SERIAL, TestPoint:TestPoint_Pad_2.0x2.0mm, F.Cu at (201.8, 134.9)
- added TP6: GND SERIAL, TestPoint:TestPoint_Pad_2.0x2.0mm, F.Cu at (201.8, 138.9)
- added U1: DSN-1504-3A, power_modules:DSN-1504-3A, F.Cu at (213.3, 66.9)
- added U2: AMS1117-3.3, Package_TO_SOT_SMD:SOT-223-3_TabPin2, F.Cu at (237.9, 80.8)
- added U3: SN75LBC179AD, SN75LBC179AD:SOIC127P599X175-8N, F.Cu at (208.5, 136.1)

Commit message: Board 3 MODBUS and servos done
Parts:
- added C8: 470n, Capacitor_SMD:C_0805_2012Metric_Pad1.18x1.45mm_HandSolder, F.Cu at (139.2, 40.3)
- moved C1 160.6 mm to (65.2, 128.5), turned to -90 degrees
- moved C5 152.7 mm to (63.0, 61.8), turned to 90 degrees
- moved U1 147.4 mm to (79.5, 128.8)
- moved U2 145.6 mm to (101.1, 130.8)
- moved TP1 135.1 mm to (94.1, 135.5)
- moved C3 131.7 mm to (94.1, 130.8), turned to 90 degrees
- moved C2 131.2 mm to (94.1, 125.7), turned to -90 degrees
- moved Q33 130.0 mm to (111.3, 33.7)
- moved Q34 129.2 mm to (111.3, 39.3)
- moved Q35 128.4 mm to (111.3, 45.0)
- moved C7 126.1 mm to (130.8, 33.2), turned to 90 degrees
- moved C4 122.6 mm to (101.2, 124.6), turned to 180 degrees
- moved D3 122.4 mm to (120.0, 133.5), turned to 180 degrees
- moved U3 122.3 mm to (132.6, 40.3), turned to 180 degrees
- moved D2 121.5 mm to (120.0, 127.5), turned to 180 degrees
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Connections:
- net /ALPHA & BETA AXIS LEVEL SHIFTING/ALF_LIM_MAX renamed /ALF_LIM_MAX
- net /ALPHA & BETA AXIS LEVEL SHIFTING/ALF_LIM_MIN renamed /ALF_LIM_MIN
- net /ALPHA & BETA AXIS LEVEL SHIFTING/BET_LIM_MAX renamed /BET_LIM_MAX
- net /ALPHA & BETA AXIS LEVEL SHIFTING/BET_LIM_MIN renamed /BET_LIM_MIN
- Q10 pad 2: Net-(Q10-S) -> /TH_ENC_B
- Q12 pad 2: Net-(Q12-S) -> /TH_LIM_MIN
- Q14 pad 2: Net-(Q14-S) -> /TH_LIM_MAX
- Q16 pad 2: Net-(Q16-S) -> /TH_HOME
- Q18 pad 2: /ALPHA & BETA AXIS LEVEL SHIFTING/ALF_ENC_A -> /ALF_ENC_A
- Q2 pad 2: /R & THETA AXIS LEVEL SHIFTING/R_LIM_MIN -> /R_LIM_MIN
- Q20 pad 2: /ALPHA & BETA AXIS LEVEL SHIFTING/ALF_ENC_B -> /ALF_ENC_B
- Q26 pad 2: /ALPHA & BETA AXIS LEVEL SHIFTING/BET_ENC_A -> /BET_ENC_A
- Q28 pad 2: /ALPHA & BETA AXIS LEVEL SHIFTING/BET_ENC_B -> /BET_ENC_B
- Q4 pad 2: /R & THETA AXIS LEVEL SHIFTING/R_LIM_MAX -> /R_LIM_MAX
- Q6 pad 2: /R & THETA AXIS LEVEL SHIFTING/R_HOME -> /R_HOME
- Q8 pad 2: Net-(Q8-S) -> /TH_ENC_A
- R22 pad 2: unconnected-(R22-Pad2) -> /R_LIM_MIN_IN
- R24 pad 1: /R & THETA AXIS LEVEL SHIFTING/R_LIM_MIN -> /R_LIM_MIN
- R25 pad 2: unconnected-(R25-Pad2) -> /R_LIM_MAX_IN
- R27 pad 1: /R & THETA AXIS LEVEL SHIFTING/R_LIM_MAX -> /R_LIM_MAX
- R28 pad 2: unconnected-(R28-Pad2) -> /R_HOME_IN
- R30 pad 1: /R & THETA AXIS LEVEL SHIFTING/R_HOME -> /R_HOME
- R31 pad 2: unconnected-(R31-Pad2) -> /TH_ENC_A_IN
- R33 pad 1: Net-(Q8-S) -> /TH_ENC_A
- R34 pad 2: unconnected-(R34-Pad2) -> /TH_ENC_B_IN
- R36 pad 1: Net-(Q10-S) -> /TH_ENC_B
- R37 pad 2: unconnected-(R37-Pad2) -> /TH_LIM_MIN_IN
- R39 pad 1: Net-(Q12-S) -> /TH_LIM_MIN
- R40 pad 2: unconnected-(R40-Pad2) -> /TH_LIM_MAX_IN
- R42 pad 1: Net-(Q14-S) -> /TH_LIM_MAX
- R43 pad 2: unconnected-(R43-Pad2) -> /TH_HOME_IN
- R45 pad 1: Net-(Q16-S) -> /TH_HOME
- R46 pad 2: /ALPHA & BETA AXIS LEVEL SHIFTING/ALF_ENC_A_IN -> /ALF_ENC_A_IN
- R48 pad 1: /ALPHA & BETA AXIS LEVEL SHIFTING/ALF_ENC_A -> /ALF_ENC_A
- R49 pad 2: /ALPHA & BETA AXIS LEVEL SHIFTING/ALF_ENC_B_IN -> /ALF_ENC_B_IN
- R51 pad 1: /ALPHA & BETA AXIS LEVEL SHIFTING/ALF_ENC_B -> /ALF_ENC_B
- R52 pad 2: /ALPHA & BETA AXIS LEVEL SHIFTING/ALF_LIM_MIN_IN -> /ALF_LIM_MIN_IN
- R55 pad 2: /ALPHA & BETA AXIS LEVEL SHIFTING/ALF_LIM_MAX_IN -> /ALF_LIM_MAX_IN
- R58 pad 2: /ALPHA & BETA AXIS LEVEL SHIFTING/BET_ENC_A_IN -> /BET_ENC_A_IN
- R60 pad 1: /ALPHA & BETA AXIS LEVEL SHIFTING/BET_ENC_A -> /BET_ENC_A
- R61 pad 2: /ALPHA & BETA AXIS LEVEL SHIFTING/BET_ENC_B_IN -> /BET_ENC_B_IN
- R63 pad 1: /ALPHA & BETA AXIS LEVEL SHIFTING/BET_ENC_B -> /BET_ENC_B
- R64 pad 2: /ALPHA & BETA AXIS LEVEL SHIFTING/BET_LIM_MIN_IN -> /BET_LIM_MIN_IN
- R67 pad 2: /ALPHA & BETA AXIS LEVEL SHIFTING/BET_LIM_MAX_IN -> /BET_LIM_MAX_IN
Routing:
- net GND: track 0.00 -> 99.8 mm, vias 0 -> 10
- net +24V: track 0.00 -> 91.5 mm, vias 0 -> 1
- net +5V: track 0.00 -> 84.0 mm, vias 0 -> 3
- net GNDS: track 0.00 -> 72.0 mm
- net +3V3: track 0.00 -> 45.8 mm
- net /ENC_PWR: track 0.00 -> 23.7 mm, vias 0 -> 3
- net /LIM_PWR: track 0.00 -> 23.7 mm, vias 0 -> 3
- net /HOME_PWR: track 0.00 -> 22.9 mm
- net +5VS: track 0.00 -> 19.7 mm
- net /END-EFFECTOR/TX_RAW: track 0.00 -> 13.1 mm, vias 0 -> 1
- net /END-EFFECTOR/RX_RAW: track 0.00 -> 11.6 mm, vias 0 -> 1
- net /R & THETA AXIS LEVEL SHIFTING/R_LIM_MIN_PG: track 0.00 -> 8.68 mm
- net /END-EFFECTOR/MODBUS_RX_N: track 0.00 -> 7.50 mm
- net /END-EFFECTOR/MODBUS_RX_P: track 0.00 -> 7.46 mm
- net /END-EFFECTOR/MODBUS_TX_N: track 0.00 -> 6.71 mm
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- added copper zone on B.Cu, net GNDS
- added copper zone on F.Cu, net GNDS
