File: Aux_boards_meta/Aux_boards_meta.kicad_pcb (KiCad board)
At the start: 2 copper layers, 21 parts, among them J1 Power out & TP, J2 ENCODER PWR SEL, J3 LIMIT-SW PWR SEL, J4 HOME-SNS PWR SEL, Q91 BSS138KJ, Q92 BSS84KJ, U1 DSN-1504-3A, U2 AMS1117-3.3

Commit message: filled out all info for meta project, starting aux boards
Parts:
- J21: renamed from J1; value Power out & TP -> PWR OUT & TP
- J22: renamed from J2; value ENCODER PWR SEL -> ENC PWR SEL
- J23: renamed from J3; value LIMIT-SW PWR SEL -> LIM PWR SEL
- J24: renamed from J4; value HOME-SNS PWR SEL -> HOM PWR SEL
- renumbered Q91 to Q1, Q92 to Q2, R91 to R4, R92 to R5, R93 to R6
Other:
- rule pad_to_mask_clearance: 0 -> 0.038
- board text added: "3v3 ENC 24V"
- board text added: "3v3 HOM 24V"
- board text added: "3v3 LIM 24V"
- board text added: "5V"
