File: Aux_boards_meta/auxboards_levelshift.kicad_sch (KiCad schematic)
At the start: 5 parts, among them Q91 BSS138KJ, Q92 BSS84KJ

Commit message: filled out all info for meta project, starting aux boards
Parts:
- renumbered Q91 to Q1, Q92 to Q2, R91 to R4, R92 to R5, R93 to R6
Changed lines of the file:
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@@
 		(dnp no)
 		(fields_autoplaced yes)
-		(property "Reference" "R91"
+		(property "Reference" "R4"
 			(at 120.65 95.25 90)
 			(effects
@@
 		)
 		(instances
-			(project "Aux_boards_meta"
-				(path "/1a58b99a-90fe-4598-8f3b-1f732cc63393/8772987c-3417-4e26-b14e-fb28636ee023"
-					(reference "R91")
+			(project "Aux_board_1"
+				(path "/066879c1-5266-4fdd-b847-a619f2624ba5/176e45ea-61c3-45df-8c32-cd3fcd81ed84"
+					(reference "R4")
+					(unit 1)
+				)
+				(path "/066879c1-5266-4fdd-b847-a619f2624ba5/d9003c61-bbad-42a3-9928-d06c6bcee20d"
+					(reference "R7")
+					(unit 1)
+				)
+				(path "/066879c1-5266-4fdd-b847-a619f2624ba5/b76ff704-f280-4a09-94a7-dedcd28f50f8"
+					(reference "R10")
+					(unit 1)
+				)
+				(path "/066879c1-5266-4fdd-b847-a619f2624ba5/58c756a1-1b91-499e-8887-9f69e8814ece"
+					(reference "R13")
+					(unit 1)
+				)
+				(path "/066879c1-5266-4fdd-b847-a619f2624ba5/b64900f0-283a-4ab8-b8b2-15a18322eadf"
+					(reference "R16")
 					(unit 1)
 				)
@@
 		(on_board yes)
 		(dnp no)
-		(property "Reference" "#PWR019"
+		(property "Reference" "#PWR023"
 			(at 138.43 116.84 0)
 			(effects
@@
 		)
 		(instances
+			(project "Aux_board_1"
+				(path "/066879c1-5266-4fdd-b847-a619f2624ba5/176e45ea-61c3-45df-8c32-cd3fcd81ed84"
+					(reference "#PWR023")
+					(unit 1)
+				)
+				(path "/066879c1-5266-4fdd-b847-a619f2624ba5/d9003c61-bbad-42a3-9928-d06c6bcee20d"
+					(reference "#PWR025")
+					(unit 1)
+				)
+				(path "/066879c1-5266-4fdd-b847-a619f2624ba5/b76ff704-f280-4a09-94a7-dedcd28f50f8"
+					(reference "#PWR027")
+					(unit 1)
+				)
+				(path "/066879c1-5266-4fdd-b847-a619f2624ba5/58c756a1-1b91-499e-8887-9f69e8814ece"
+					(reference "#PWR029")
+					(unit 1)
+				)
+			)
 			(project "Aux_boards_meta"
 				(path "/1a58b99a-90fe-4598-8f3b-1f732cc63393/8772987c-3417-4e26-b14e-fb28636ee023"
-					(reference "#PWR019")
+					(reference "#PWR023")
 					(unit 1)
 				)
@@
 		(dnp no)
 		(fields_autoplaced yes)
-		(property "Reference" "R92"
+		(property "Reference" "R5"
 			(at 140.97 83.8199 0)
 			(effects
@@
 		)
 		(instances
-			(project "Aux_boards_meta"
-				(path "/1a58b99a-90fe-4598-8f3b-1f732cc63393/8772987c-3417-4e26-b14e-fb28636ee023"
-					(reference "R92")
+			(project "Aux_board_1"
+				(path "/066879c1-5266-4fdd-b847-a619f2624ba5/176e45ea-61c3-45df-8c32-cd3fcd81ed84"
+					(reference "R5")
+					(unit 1)
+				)
+				(path "/066879c1-5266-4fdd-b847-a619f2624ba5/d9003c61-bbad-42a3-9928-d06c6bcee20d"
+					(reference "R8")
+					(unit 1)
+				)
+				(path "/066879c1-5266-4fdd-b847-a619f2624ba5/b76ff704-f280-4a09-94a7-dedcd28f50f8"
+					(reference "R11")
+					(unit 1)
+				)
+				(path "/066879c1-5266-4fdd-b847-a619f2624ba5/58c756a1-1b91-499e-8887-9f69e8814ece"
+					(reference "R14")
+					(unit 1)
+				)
+				(path "/066879c1-5266-4fdd-b847-a619f2624ba5/b64900f0-283a-4ab8-b8b2-15a18322eadf"
+					(reference "R17")
 					(unit 1)
 				)
@@
 		(dnp no)
 		(fields_autoplaced yes)
-		(property "Reference" "Q92"
+		(property "Reference" "Q2"
 			(at 158.75 90.1699 0)
 			(effects
@@
 		)
 		(instances
-			(project "Aux_boards_meta"
-				(path "/1a58b99a-90fe-4598-8f3b-1f732cc63393/8772987c-3417-4e26-b14e-fb28636ee023"
-					(reference "Q92")
+			(project "Aux_board_1"
+				(path "/066879c1-5266-4fdd-b847-a619f2624ba5/176e45ea-61c3-45df-8c32-cd3fcd81ed84"
+					(reference "Q2")
+					(unit 1)
+				)
+				(path "/066879c1-5266-4fdd-b847-a619f2624ba5/d9003c61-bbad-42a3-9928-d06c6bcee20d"
+					(reference "Q4")
+					(unit 1)
+				)
+				(path "/066879c1-5266-4fdd-b847-a619f2624ba5/b76ff704-f280-4a09-94a7-dedcd28f50f8"
+					(reference "Q6")
+					(unit 1)
+				)
+				(path "/066879c1-5266-4fdd-b847-a619f2624ba5/58c756a1-1b91-499e-8887-9f69e8814ece"
+					(reference "Q8")
+					(unit 1)
+				)
+				(path "/066879c1-5266-4fdd-b847-a619f2624ba5/b64900f0-283a-4ab8-b8b2-15a18322eadf"
+					(reference "Q10")
 					(unit 1)
 				)
@@
 		(dnp no)
 		(fields_autoplaced yes)
-		(property "Reference" "R93"
+		(property "Reference" "R6"
 			(at 157.48 102.8699 0)
 			(effects
@@
 		)
 		(instances
-			(project "Aux_boards_meta"
-				(path "/1a58b99a-90fe-4598-8f3b-1f732cc63393/8772987c-3417-4e26-b14e-fb28636ee023"
-					(reference "R93")
+			(project "Aux_board_1"
+				(path "/066879c1-5266-4fdd-b847-a619f2624ba5/176e45ea-61c3-45df-8c32-cd3fcd81ed84"
+					(reference "R6")
+					(unit 1)
+				)
+				(path "/066879c1-5266-4fdd-b847-a619f2624ba5/d9003c61-bbad-42a3-9928-d06c6bcee20d"
+					(reference "R9")
+					(unit 1)
+				)
+				(path "/066879c1-5266-4fdd-b847-a619f2624ba5/b76ff704-f280-4a09-94a7-dedcd28f50f8"
+					(reference "R12")
+					(unit 1)
+				)
+				(path "/066879c1-5266-4fdd-b847-a619f2624ba5/58c756a1-1b91-499e-8887-9f69e8814ece"
+					(reference "R15")
+					(unit 1)
+				)
+				(path "/066879c1-5266-4fdd-b847-a619f2624ba5/b64900f0-283a-4ab8-b8b2-15a18322eadf"
+					(reference "R18")
 					(unit 1)
 				)
@@
 		(dnp no)
 		(fields_autoplaced yes)
-		(property "Reference" "Q91"
+		(property "Reference" "Q1"
 			(at 142.24 100.3299 0)
 			(effects
@@
 		)
 		(instances
-			(project "Aux_boards_meta"
-				(path "/1a58b99a-90fe-4598-8f3b-1f732cc63393/8772987c-3417-4e26-b14e-fb28636ee023"
-					(reference "Q91")
+			(project "Aux_board_1"
+				(path "/066879c1-5266-4fdd-b847-a619f2624ba5/176e45ea-61c3-45df-8c32-cd3fcd81ed84"
+					(reference "Q1")
+					(unit 1)
+				)
+				(path "/066879c1-5266-4fdd-b847-a619f2624ba5/d9003c61-bbad-42a3-9928-d06c6bcee20d"
+					(reference "Q3")
+					(unit 1)
+				)
+				(path "/066879c1-5266-4fdd-b847-a619f2624ba5/b76ff704-f280-4a09-94a7-dedcd28f50f8"
+					(reference "Q5")
+					(unit 1)
+				)
+				(path "/066879c1-5266-4fdd-b847-a619f2624ba5/58c756a1-1b91-499e-8887-9f69e8814ece"
+					(reference "Q7")
+					(unit 1)
+				)
+				(path "/066879c1-5266-4fdd-b847-a619f2624ba5/b64900f0-283a-4ab8-b8b2-15a18322eadf"
+					(reference "Q9")
 					(unit 1)
 				)
@@
 		(dnp no)
 		(fields_autoplaced yes)
-		(property "Reference" "#PWR018"
+		(property "Reference" "#PWR022"
 			(at 138.43 80.01 0)
 			(effects
@@
 		)
 		(instances
+			(project "Aux_board_1"
+				(path "/066879c1-5266-4fdd-b847-a619f2624ba5/176e45ea-61c3-45df-8c32-cd3fcd81ed84"
+					(reference "#PWR022")
+					(unit 1)
+				)
+				(path "/066879c1-5266-4fdd-b847-a619f2624ba5/d9003c61-bbad-42a3-9928-d06c6bcee20d"
+					(reference "#PWR024")
+					(unit 1)
+				)
+				(path "/066879c1-5266-4fdd-b847-a619f2624ba5/b76ff704-f280-4a09-94a7-dedcd28f50f8"
+					(reference "#PWR026")
+					(unit 1)
+				)
+				(path "/066879c1-5266-4fdd-b847-a619f2624ba5/58c756a1-1b91-499e-8887-9f69e8814ece"
+					(reference "#PWR028")
+					(unit 1)
+				)
+			)
 			(project "Aux_boards_meta"
 				(path "/1a58b99a-90fe-4598-8f3b-1f732cc63393/8772987c-3417-4e26-b14e-fb28636ee023"
-					(reference "#PWR018")
-					(unit 1)
-				)
+					(reference "#PWR022")
+					(unit 1)
+				)
