File: Aux_boards_meta/auxboards_power.kicad_sch (KiCad schematic)
At the start: 16 parts, among them J1 Power out & TP, J2 ENCODER PWR SEL, J3 LIMIT-SW PWR SEL, J4 HOME-SNS PWR SEL, U1 DSN-1504-3A, U2 AMS1117-3.3

Commit message: filled out all info for meta project, starting aux boards
Parts:
- J1: value Power out & TP -> PWR OUT & TP
- J2: value ENCODER PWR SEL -> ENC PWR SEL
- J3: value LIMIT-SW PWR SEL -> LIM PWR SEL
- J4: value HOME-SNS PWR SEL -> HOM PWR SEL
